File: analog.kicad_sch (KiCad schematic)
At the start: 50 parts, among them J8 Sensor harness, J9 Spare diff in, U8 ADS1115 (0x48), U9 ADS1115 (0x49)

Commit message: Route, audit and document the carrier; verify every part number against the catalogue
Ordering is the point of this pass, so the part numbers came first. Every
LCSC number on the board was opened and read -- manufacturer part, package,
and the parameter that decides whether it is the right part. That found:

  C2148396 for the MCP2518FD    is an 18.7k resistor, out of stock -> C626759
  C255909  for a 40 MHz crystal is a 16 MHz crystal              -> C5186937
  C157966  for a JST PH 10-way  is a JST XH 9-way, 2.5 mm pitch  -> C158038

Three of the five numbers introduced last sitting were wrong, and all three
were plausible enough that the BOM exported clean. docs/PARTS.md records the
lot, including that LCSC's own listing for the microSD socket claims it has
no card-detect switch -- it has one, and the schematic is right.

Two footprints would not have soldered: both polyfuses are 1812 parts sitting
on a 1206 land, inherited from the parent board where nothing had ever
compared a part's package against its footprint. And the generic-passive
table was keyed on value alone, so the 1206 positions added last sitting
would have ordered 0805 parts -- right resistance, wrong footprint, every
board. It is keyed on (value, package) now and returns nothing rather than
guessing, so an unmatched line has no part number and somebody has to look.

Several values moved to match what is actually stocked: the power-fail
divider to 43k/18k (same trip point to 2 mV, both stocked 1 % parts), the
K-line series and pull-up to 20 R and 750 R, and the supercap charge resistor
from 22 R to 100 R -- 22 R put 1 W into a 250 mW part for the first several
seconds of every power-up.

Two real defects, both found by tools rather than by reading:

  - The hold-up Schottky was BACKWARDS. Reversed it shorts out the inrush
    limiter and blocks the discharge, so the supercap bank could never hold
    the rail up and the whole hold-up circuit was inert. audit_polarity found
    it once its expectat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
Parts:
- removed J8: Sensor harness, Connector_JST:JST_PH_B10B-PH-K_1x10_P2.00mm_Vertical, symbol Connector_Generic:Conn_01x10
- added J10: Spare diff in, Connector_PinHeader_2.54mm:PinHeader_1x04_P2.54mm_Vertical, symbol Connector_Generic:Conn_01x04
- C25: value 100nF -> 470nF; Note Ch1 anti-alias / ADC charge reservoir -> Ch1 anti-alias. 470nF, not the 100nF this inherited: source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; Voltage 16V -> 50V
- C26: value 100nF -> 470nF; Note Ch2 anti-alias / ADC charge reservoir -> Ch2 anti-alias. 470nF, not the 100nF this inherited: source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; Voltage 16V -> 50V
- C27: value 100nF -> 470nF; Note Ch3 anti-alias / ADC charge reservoir -> Ch3 anti-alias. 470nF, not the 100nF this inherited: source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; Voltage 16V -> 50V
- C28: value 100nF -> 470nF; Note Ch4 anti-alias / ADC charge reservoir -> Ch4 anti-alias. 470nF, not the 100nF this inherited: source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; Voltage 16V -> 50V
- C29: value 100nF -> 470nF; Note Matches the channels' filter -> Matches the channels' filter, and this one is not cosmetic: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; Voltage 16V -> 50V
- J9: value Spare diff in -> Sensor harness; footprint Connector_PinHeader_2.54mm:PinHeader_1x04_P2.54mm_Vertical -> Connector_JST:JST_PH_B10B-PH-K_1x10_P2.00mm_Vertical; symbol Connector_Generic:Conn_01x04 -> Connector_Generic:Conn_01x10; MPN (none) -> JST B10B-PH-K-S(LF)(SN); Note The second ADC's unused pair, brought out raw -- 0-3.3V onl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 -> Two 5V excitation pins, two Kelvin sense-ground pins, two c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
Connections:
- net +5VS: now also J9.1 (Pin_1), J9.2 (Pin_2)
- net AGND_SENSE: now also J10.3 (Pin_3); no longer J9.3 (Pin_3)
- net AIN1_IN: now also J9.3 (Pin_3)
- net AIN2_IN: now also J9.4 (Pin_4)
- net AIN3_IN: now also J9.7 (Pin_7)
- net AIN4_IN: now also J9.8 (Pin_8)
- net AIN_SP1: now also J10.1 (Pin_1); no longer J9.1 (Pin_1)
- net AIN_SP2: now also J10.2 (Pin_2); no longer J9.2 (Pin_2)
- net GND: now also J9.10 (Pin_10), J9.9 (Pin_9), J10.4 (Pin_4); no longer J9.4 (Pin_4)
- net SENS_RTN: now also J9.5 (Pin_5), J9.6 (Pin_6)
Changed lines of the file:
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@@
   (symbol (lib_id "Connector_Generic:Conn_01x10") (at 46.99 27.94 0) (unit 1)
     (in_bom yes) (on_board yes) (dnp no)
-    (property "Reference" "J8" (at 46.99 15.78 0)
+    (property "Reference" "J9" (at 46.99 15.78 0)
       (effects (font (size 1.27 1.27)) )
     )
@@
     (instances
       (project "esp32s3-can-sd-logger"
-        (path "/3276c6e6-7085-5954-8442-c6cef7eab316/61f1fdfe-4c14-50c2-a034-e9770d48c32f" (reference "J8") (unit 1))
+        (path "/3276c6e6-7085-5954-8442-c6cef7eab316/61f1fdfe-4c14-50c2-a034-e9770d48c32f" (reference "J9") (unit 1))
       )
     )
@@
       (effects (font (size 1.27 1.27)) (justify left) )
     )
-    (property "Value" "100nF" (at 93.98 85.6 0)
+    (property "Value" "470nF" (at 93.98 85.6 0)
       (effects (font (size 1.27 1.27)) (justify left) )
     )
@@
       (effects (font (size 1.27 1.27)) (justify left) hide)
     )
-    (property "Voltage" "16V" (at 93.98 85.6 0)
-      (effects (font (size 1.27 1.27)) (justify left) hide)
-    )
-    (property "Note" "Ch1 anti-alias / ADC charge reservoir" (at 93.98 85.6 0)
+    (property "Voltage" "50V" (at 93.98 85.6 0)
+      (effects (font (size 1.27 1.27)) (justify left) hide)
+    )
+    (property "Note" "Ch1 anti-alias. 470nF, not the 100nF this inherited: source impedance here is (1k+10k)||2.21k = 1.84k, so 100nF puts the corner at 865 Hz -- above the 430 Hz Nyquist of the ADS1115 at 860 SPS, and well above anything the ESP32's own SAR ADC can sample cleanly. That was survivable while 0-5 V was the default range (261 Hz) and became the only behaviour when the range jumpers went. 470nF gives 184 Hz, which still passes anything a wideband does and stops engine noise folding into the log" (at 93.98 85.6 0)
       (effects (font (size 1.27 1.27)) (justify left) hide)
     )
@@
       (effects (font (size 1.27 1.27)) (justify left) )
     )
-    (property "Value" "100nF" (at 93.98 136.4 0)
+    (property "Value" "470nF" (at 93.98 136.4 0)
       (effects (font (size 1.27 1.27)) (justify left) )
     )
@@
       (effects (font (size 1.27 1.27)) (justify left) hide)
     )
-    (property "Voltage" "16V" (at 93.98 136.4 0)
-      (effects (font (size 1.27 1.27)) (justify left) hide)
-    )
-    (property "Note" "Ch2 anti-alias / ADC charge reservoir" (at 93.98 136.4 0)
+    (property "Voltage" "50V" (at 93.98 136.4 0)
+      (effects (font (size 1.27 1.27)) (justify left) hide)
+    )
+    (property "Note" "Ch2 anti-alias. 470nF, not the 100nF this inherited: source impedance here is (1k+10k)||2.21k = 1.84k, so 100nF puts the corner at 865 Hz -- above the 430 Hz Nyquist of the ADS1115 at 860 SPS, and well above anything the ESP32's own SAR ADC can sample cleanly. That was survivable while 0-5 V was the default range (261 Hz) and became the only behaviour when the range jumpers went. 470nF gives 184 Hz, which still passes anything a wideband does and stops engine noise folding into the log" (at 93.98 136.4 0)
       (effects (font (size 1.27 1.27)) (justify left) hide)
     )
@@
       (effects (font (size 1.27 1.27)) (justify left) )
     )
-    (property "Value" "100nF" (at 93.98 187.2 0)
+    (property "Value" "470nF" (at 93.98 187.2 0)
       (effects (font (size 1.27 1.27)) (justify left) )
     )
@@
       (effects (font (size 1.27 1.27)) (justify left) hide)
     )
-    (property "Voltage" "16V" (at 93.98 187.2 0)
-      (effects (font (size 1.27 1.27)) (justify left) hide)
-    )
-    (property "Note" "Ch3 anti-alias / ADC charge reservoir" (at 93.98 187.2 0)
+    (property "Voltage" "50V" (at 93.98 187.2 0)
+      (effects (font (size 1.27 1.27)) (justify left) hide)
+    )
+    (property "Note" "Ch3 anti-alias. 470nF, not the 100nF this inherited: source impedance here is (1k+10k)||2.21k = 1.84k, so 100nF puts the corner at 865 Hz -- above the 430 Hz Nyquist of the ADS1115 at 860 SPS, and well above anything the ESP32's own SAR ADC can sample cleanly. That was survivable while 0-5 V was the default range (261 Hz) and became the only behaviour when the range jumpers went. 470nF gives 184 Hz, which still passes anything a wideband does and stops engine noise folding into the log" (at 93.98 187.2 0)
       (effects (font (size 1.27 1.27)) (justify left) hide)
     )
@@
       (effects (font (size 1.27 1.27)) (justify left) )
     )
-    (property "Value" "100nF" (at 93.98 239.27 0)
+    (property "Value" "470nF" (at 93.98 239.27 0)
       (effects (font (size 1.27 1.27)) (justify left) )
     )
@@
       (effects (font (size 1.27 1.27)) (justify left) hide)
     )
-    (property "Voltage" "16V" (at 93.98 239.27 0)
-      (effects (font (size 1.27 1.27)) (justify left) hide)
-    )
-    (property "Note" "Ch4 anti-alias / ADC charge reservoir" (at 93.98 239.27 0)
+    (property "Voltage" "50V" (at 93.98 239.27 0)
+      (effects (font (size 1.27 1.27)) (justify left) hide)
+    )
+    (property "Note" "Ch4 anti-alias. 470nF, not the 100nF this inherited: source impedance here is (1k+10k)||2.21k = 1.84k, so 100nF puts the corner at 865 Hz -- above the 430 Hz Nyquist of the ADS1115 at 860 SPS, and well above anything the ESP32's own SAR ADC can sample cleanly. That was survivable while 0-5 V was the default range (261 Hz) and became the only behaviour when the range jumpers went. 470nF gives 184 Hz, which still passes anything a wideband does and stops engine noise folding into the log" (at 93.98 239.27 0)
       (effects (font (size 1.27 1.27)) (justify left) hide)
     )
@@
       (effects (font (size 1.27 1.27)) )
     )
-    (property "Value" "100nF" (at 158.75 60.42 270)
+    (property "Value" "470nF" (at 158.75 60.42 270)
       (effects (font (size 1.27 1.27)) )
     )
@@
       (effects (font (size 1.27 1.27)) hide)
     )
-    (property "Voltage" "16V" (at 158.75 60.42 270)
-      (effects (font (size 1.27 1.27)) hide)
-    )
-    (property "Note" "Matches the channels' filter" (at 158.75 60.42 270)
+    (property "Voltage" "50V" (at 158.75 60.42 270)
+      (effects (font (size 1.27 1.27)) hide)
+    )
+    (property "Note" "Matches the channels' filter, and this one is not cosmetic: the ground correction is the difference of two attenuators, so if their corner frequencies differ the subtraction leaves a phase residue on every transient. Same value, same dielectric, same part number" (at 158.75 60.42 270)
       (effects (font (size 1.27 1.27)) hide)
     )
@@
   (symbol (lib_id "Connector_Generic:Conn_01x04") (at 240.03 20.32 0) (unit 1)
     (in_bom yes) (on_board yes) (dnp no)
-    (property "Reference" "J9" (at 240.03 15.78 0)
+    (property "Reference" "J10" (at 240.03 15.78 0)
       (effects (font (size 1.27 1.27)) )
     )
@@
     (instances
       (project "esp32s3-can-sd-logger"
-        (path "/3276c6e6-7085-5954-8442-c6cef7eab316/61f1fdfe-4c14-50c2-a034-e9770d48c32f" (reference "J9") (unit 1))
-      )
-    )
+        (path "/3276c6e6-7085-5954-8442-c6cef7eab316/61f1fdfe-4c14-50c2-a034-e9770d48c32f" (reference "J10") (unit 1))
+      )
+    )

Commit message: Implement the cost reductions: 1% dividers and a 0.33 F bank -- $18.29 to $13.87
Two of the three changes from docs/COST.md. The third was dropped once I
checked it properly, which is the more interesting half of this commit.

PRECISION RESISTORS TO 1%, saving $2.62 measured. Fifteen 0.1% parts cost
$2.68 -- more than the CAN controller -- to tighten a divider whose error the
ADS1115's own +/-0.30% gain spec already dominates. Absolute scale has to be
calibrated whatever the tolerance, and the thing calibration cannot fix, the
match between the signal chain and the return attenuator, is fine at 1%: a
300 mV chassis offset leaves 6 mV instead of 0.6 mV, both negligible against
the 300 mV being removed.

The lower leg went 2.21k -> 2.2k with it, because E96 values do not exist in
the 1% jellybean library. That is a happy accident: 2.2/13.2 is exactly 1/6,
so DIVIDER_GAIN is a round 6.0000 instead of 5.9774.

HOLD-UP BANK 1 F -> 0.33 F per cell, saving roughly $1.80. 1 F bought 2500 ms
that nothing needs -- the parent board shipped 127 ms and that was judged
adequate, a healthy card flushes in 18 ms, and the worst stall the firmware
studies model is 500 ms. 0.33 F gives 825 ms shed, six times the parent's
margin and still 65% clear of that worst case. The budgets in fwsim, studies
11 and 12 and their sweep ranges all move with it.

THE microSD SWAP IS NOT DONE, and the $1.06 I quoted for it was arithmetic
against a part I could not verify. Those $0.04 sockets are house parts whose
only drawing is a scanned PDF with no extractable dimensions, so the land
pattern cannot be checked -- and shipping an unverified footprint on five
boards to save a dollar is not a trade this project should make. The
verifiable alternatives are worse than the search suggested: the Molex
47219-2001 with a KiCad footprint is $0.63 against the Hirose's $1.12, so the
honest saving is $0.49, and it costs the card-detect signal and swaps a
push-pull for a hinged lid. The Hirose stays. COST.md recor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
Parts:
- R37: Note Ch1 series/fault-current limit; 0.1% thin film -- it is ins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 -> Ch1 series/fault-current limit. 1%, not the 0.1% thin film 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; Tolerance 0.1% -> (none)
- R39: Note Ch1 divider upper leg, 0.1% thin film for AFR-grade accuracy -> Ch1 divider upper leg; Tolerance 0.1% -> (none)
- R40: value 2.21k -> 2.2k; Note Ch1 divider lower leg. 2.21/13.21 = 0.1673, so 16.0 V in gi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 -> Ch1 divider lower leg. 2.2/13.2 = exactly 1/6, so 16.0 V in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; Tolerance 0.1% -> (none)
- R41: Note Ch2 series/fault-current limit; 0.1% thin film -- it is ins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 -> Ch2 series/fault-current limit. 1%, not the 0.1% thin film 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; Tolerance 0.1% -> (none)
- R43: Note Ch2 divider upper leg, 0.1% thin film for AFR-grade accuracy -> Ch2 divider upper leg; Tolerance 0.1% -> (none)
- R44: value 2.21k -> 2.2k; Note Ch2 divider lower leg. 2.21/13.21 = 0.1673, so 16.0 V in gi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 -> Ch2 divider lower leg. 2.2/13.2 = exactly 1/6, so 16.0 V in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; Tolerance 0.1% -> (none)
- R45: Note Ch3 series/fault-current limit; 0.1% thin film -- it is ins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 -> Ch3 series/fault-current limit. 1%, not the 0.1% thin film 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; Tolerance 0.1% -> (none)
- R47: Note Ch3 divider upper leg, 0.1% thin film for AFR-grade accuracy -> Ch3 divider upper leg; Tolerance 0.1% -> (none)
- R48: value 2.21k -> 2.2k; Note Ch3 divider lower leg. 2.21/13.21 = 0.1673, so 16.0 V in gi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 -> Ch3 divider lower leg. 2.2/13.2 = exactly 1/6, so 16.0 V in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; Tolerance 0.1% -> (none)
- R49: Note Ch4 series/fault-current limit; 0.1% thin film -- it is ins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 -> Ch4 series/fault-current limit. 1%, not the 0.1% thin film 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; Tolerance 0.1% -> (none)
- R51: Note Ch4 divider upper leg, 0.1% thin film for AFR-grade accuracy -> Ch4 divider upper leg; Tolerance 0.1% -> (none)
- R52: value 2.21k -> 2.2k; Note Ch4 divider lower leg. 2.21/13.21 = 0.1673, so 16.0 V in gi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 -> Ch4 divider lower leg. 2.2/13.2 = exactly 1/6, so 16.0 V in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; Tolerance 0.1% -> (none)
- R53, R54: Tolerance 0.1% -> (none)
- R55: value 2.21k -> 2.2k; Note Matches the channels' lower leg. Same value, same 0.1%% par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 -> Matches the channels' lower leg. Same value, same part, sam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; Tolerance 0.1% -> (none)

Commit message: Precision where it changes the answer: 0.1% on the two gain-setting resistors
Walking back half of the previous commit, because its argument depended on a
calibration step that is not going to happen. All-1% dividers are only
equivalent to 0.1% if somebody measures each channel against a known voltage
and stores a constant; without that they are 1.67% worst case against 0.167%.

But going straight back to fifteen 0.1% parts would have been the wrong
correction. Gain is Rlow/(Rser+Rup+Rlow), so each resistor moves it in
proportion to its share of the total:

    1k series    0.076 -> 0.076% of gain per 1% of tolerance
    10k upper    0.758 -> 0.758%
    2.21k lower  0.833 -> 0.833%

The series resistor is TEN TIMES less sensitive than the other two, and it
was the most expensive 0.1% part on the board at $0.30 against $0.19 and
$0.05. So it stays 1% and the two that set the ratio go back to 0.1%.

That lands the divider at 0.235% worst case, just under the ADS1115's own
0.30% maximum gain error -- the point past which spending more buys nothing --
and it needs no calibration. $1.21 a board against $2.68 for all-0.1% and
$0.05 for all-1%.

Board is $15.02 against the $18.29 it started at, an 18% cut rather than the
24% the previous commit claimed. DIVIDER_GAIN returns to 5.9774 and the ratio
is 2.21/13.21 again; the exact-1/6 was a nicety of the all-1% build, not a
requirement.

Also adds gen/audit_schematic.py, which measures two things nothing else
looks at: text printed on top of other text, and symbols connected only by
net label with no wire attached. It found its own first bug immediately --
counting the lib_symbols block, where every library definition carries
Reference and Value properties at identical coordinates, as 187 collisions
that do not exist on the drawing.

Verification unchanged: ERC clean, DRC 0 violations 0 unconnected, 50/50
firmware checks, 17/17 mutations, ngspice clean, docs audit clean.
Parts:
- R37: Note Ch1 series/fault-current limit. 1%, not the 0.1% thin film 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 -> Ch1 series/fault-current limit. 1%, and the ONLY 1% part in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
- R39: Note Ch1 divider upper leg -> Ch1 divider upper leg. 0.1%: this and the lower leg set the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; Tolerance (none) -> 0.1%
- R40: value 2.2k -> 2.21k; Note Ch1 divider lower leg. 2.2/13.2 = exactly 1/6, so 16.0 V in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 -> Ch1 divider lower leg, and the most gain-sensitive part in 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; Tolerance (none) -> 0.1%
- R41: Note Ch2 series/fault-current limit. 1%, not the 0.1% thin film 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 -> Ch2 series/fault-current limit. 1%, and the ONLY 1% part in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
- R43: Note Ch2 divider upper leg -> Ch2 divider upper leg. 0.1%: this and the lower leg set the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; Tolerance (none) -> 0.1%
- R44: value 2.2k -> 2.21k; Note Ch2 divider lower leg. 2.2/13.2 = exactly 1/6, so 16.0 V in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 -> Ch2 divider lower leg, and the most gain-sensitive part in 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; Tolerance (none) -> 0.1%
- R45: Note Ch3 series/fault-current limit. 1%, not the 0.1% thin film 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 -> Ch3 series/fault-current limit. 1%, and the ONLY 1% part in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
- R47: Note Ch3 divider upper leg -> Ch3 divider upper leg. 0.1%: this and the lower leg set the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; Tolerance (none) -> 0.1%
- R48: value 2.2k -> 2.21k; Note Ch3 divider lower leg. 2.2/13.2 = exactly 1/6, so 16.0 V in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 -> Ch3 divider lower leg, and the most gain-sensitive part in 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; Tolerance (none) -> 0.1%
- R49: Note Ch4 series/fault-current limit. 1%, not the 0.1% thin film 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 -> Ch4 series/fault-current limit. 1%, and the ONLY 1% part in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
- R51: Note Ch4 divider upper leg -> Ch4 divider upper leg. 0.1%: this and the lower leg set the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; Tolerance (none) -> 0.1%
- R52: value 2.2k -> 2.21k; Note Ch4 divider lower leg. 2.2/13.2 = exactly 1/6, so 16.0 V in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 -> Ch4 divider lower leg, and the most gain-sensitive part in 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; Tolerance (none) -> 0.1%
- R54: Tolerance (none) -> 0.1%
- R55: value 2.2k -> 2.21k; Tolerance (none) -> 0.1%
