File: can.kicad_sch (KiCad schematic)
At the start: 13 parts, among them U12 TJA1051T/3

Commit message: Re-scope the fork as a carrier board: no power section, differential analog, K-line
The shield idea does not survive measurement. Component courtyard on the
parent is 3052 mm2 over an 84 x 100 board -- 36% packing, not the 50% I had
been estimating -- and a DevKitC-1 is 63 x 25.5 = 1607 mm2. The parts alone
were 1.4x the whole dev board. So this is a carrier the dev board plugs into,
not a shield that fits on top of one.

Power section deleted entirely. It was 1746 mm2, 57% of the board, for two
rails the DevKitC-1 already makes from its USB-C. Gone: both LM5164 bucks and
everything around them, the LM74700 ideal diode, the reverse-battery FET, the
three electrolytic cans, the 12 V input, and the sensor-rail load switch.
Both rails are now inputs, taken up through the sockets -- which reverses the
earlier "feed 5 V only" rule, because there is no longer a second regulator
to parallel against.

Hold-up is a supercapacitor, not electrolytics. The first sizing was wrong:
energy goes as V-squared and the usable window at 5 V is 4.2 -> 3.6 V, so
2000 uF buys 12.5 ms, not the ~50 ms claimed. 0.5 F over the same window is
2.5 s, in less area than one of the 100 V cans it replaces. Low-ESR
cylindrical cells specifically -- coin EDLCs are 30-200 ohm and cannot source
120 mA at all.

Analog runs differentially. The board is grounded twice now, through the
sensor loom and through USB by way of a charger elsewhere in the car, and a
few hundred mV of chassis drop is 6% of a 0-5 V channel -- which makes the
0.1% dividers pointless. The correction has to be at the divider, not the
ADC, so the sensor ground comes back as a Kelvin wire through a matched
attenuator. Two ADS1115s, because one MUX only offers three channels against
a shared negative.

K-line added, discrete rather than an L9637D: that part's TXD threshold is
0.7*VCC = 3.5 V and a 3.3 V GPIO cannot meet it. Low-side 2N7002, clamped
22k/10k receiver, optional ISO 9141 tester pull-up on a jumper.

Pin map regrouped by boa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
Parts:
- removed C35, C36: 100nF, Capacitor_SMD:C_0805_2012Metric, symbol Device:C
- removed C37: 4.7nF, Capacitor_SMD:C_0805_2012Metric, symbol Device:C
- removed L3: 51uH, esp32autosport:L_CommonMode_TDK_ACT45B, symbol Device:L_Coupled
- removed R54: 10k, Resistor_SMD:R_0805_2012Metric, symbol Device:R
- removed R55, R56: 60.4, Resistor_SMD:R_0805_2012Metric, symbol Device:R
- removed TP11: CAN_L, TestPoint:TestPoint_Pad_D1.5mm, symbol Connector:TestPoint
- removed U12: TJA1051T/3, Package_SO:SOIC-8_3.9x4.9mm_P1.27mm, symbol Interface_CAN_LIN:TJA1051T-3
- added C15, C16: 100nF, Capacitor_SMD:C_0805_2012Metric, symbol Device:C
- added C17: 4.7nF, Capacitor_SMD:C_0805_2012Metric, symbol Device:C
- added D5: SMAJ26CA, Diode_SMD:D_SMA, symbol Device:D_TVS
- added D8: BAT54S, Package_TO_SOT_SMD:SOT-23, symbol Device:D_Schottky_Dual_Series_AKC
- added JP2: KPU (default OFF), Jumper:SolderJumper-2_P1.3mm_Open_Pad1.0x1.5mm, symbol Jumper:SolderJumper_2_Open
- added L1: 51uH, esp32autosport:L_CommonMode_TDK_ACT45B, symbol Device:L_Coupled
- added Q3: 2N7002, Package_TO_SOT_SMD:SOT-23, symbol Transistor_FET:Q_NMOS_GSD
- added R28, R31, R35: 10k, Resistor_SMD:R_0805_2012Metric, symbol Device:R
- added R29, R30: 60.4, Resistor_SMD:R_0805_2012Metric, symbol Device:R
- added R32: 100k, Resistor_SMD:R_0805_2012Metric, symbol Device:R
- added R33: 33, Resistor_SMD:R_1206_3216Metric, symbol Device:R
- added R34: 22k, Resistor_SMD:R_0805_2012Metric, symbol Device:R
- added R36: 510, Resistor_SMD:R_1206_3216Metric, symbol Device:R
- added TP8: CAN_H, TestPoint:TestPoint_Pad_D1.5mm, symbol Connector:TestPoint
- added TP9: CAN_L, TestPoint:TestPoint_Pad_D1.5mm, symbol Connector:TestPoint
- added U5: TJA1051T/3, Package_SO:SOIC-8_3.9x4.9mm_P1.27mm, symbol Interface_CAN_LIN:TJA1051T-3
- D6: Note Bidirectional bus clamp -> (none)
- D7: Note (none) -> K-line harness clamp. Same part as the two CAN clamps, so i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
- TP10: value CAN_H -> K_LINE
Connections:
- net +3V3: now also C16.1, D8.2 (K), U5.5 (VIO)
- net +5V: now also C15.1, U5.3 (VCC)
- net CANH_T: now also L1.1, U5.7 (CANH)
- net CANL_T: now also L1.3, U5.6 (CANL)
- net CAN_H: now also D5.1 (A1), L1.2, TP8.1; no longer D6.1 (A1), TP10.1
- net CAN_L: now also D6.1 (A1), L1.4, R30.2, TP9.1; no longer D7.1 (A1)
- net CAN_RX: now also U5.4 (RXD)
- net CAN_S: now also R28.1, U5.8 (S)
- net CAN_SPLIT: now also C17.1, R29.2, R30.1
- net CAN_TX: now also U5.1 (TXD)
- net GND: now also C15.2, C16.2, C17.2, D5.2 (A2), D8.1 (A), Q3.2 (S), R28.2, R32.2, R35.2, U5.2 (GND)
- net TERM_A: now also R29.1
- new net K_LINE: D7.1 (A1), R33.2, R34.1, R36.2, TP10.1
- new net K_PU: JP2.2 (B), R36.1
- new net K_RX: D8.3 (common), R34.2, R35.1
- new net K_TX: R31.1
- new net K_TX_D: Q3.3 (D), R33.1
- new net K_TX_G: Q3.1 (G), R31.2, R32.1
- new net OBD_VBAT_F: JP2.1 (A)
Other:
- moved on the sheet: D6, D7, TP10

Commit message: Second CAN bus, single analog range, and three placement bugs the render caught
TWO CAN BUSES AT ONCE NEEDS A SECOND CONTROLLER. The ESP32-S3 has exactly
one TWAI peripheral. Two transceivers on it would give a bus you can pick at
runtime through the GPIO matrix, never two live at once, and the point of a
second bus is watching the powertrain and the body bus together. So the
second channel is an MCP2518FD on SPI (SOIC-14, KiCad ships the pin-compatible
MCP2517FD symbol) with its own 40 MHz crystal, its own TJA1051 -- same part
as CAN 1, so two positions on one BOM line -- choke, split termination and
clamps.

That cost five pins against two spare. The three came from dropping the
microSD to 1-bit SDMMC, which measurement says is free: the busiest case this
logger will see is ~128 kB/s against 1-bit's ~1500 kB/s, and bus width does
not touch the card's internal write stall, which is the only thing the
hold-up budget is actually sized around. The card keeps its D1/D2/D3
pull-ups because a card samples DAT3 at power-up and drops into SPI mode if
it finds it low -- they simply stop at the socket now.

Jumpers on the aux harness pins pick K-line or the second CAN pair, because
those two genuinely cannot share a wire: K-line idles at battery voltage and
a CAN transceiver biases its bus to 2.5 V. The clamps sit ahead of the
jumpers so the protection is the same either way, which also let the K-line
drop its own TVS. Default is K-line, which is what an R53 wants.

ANALOG DOWN TO ONE RANGE. The bypass and range-select jumpers are gone --
twelve jumpers and four resistors -- and every channel is a fixed 2.21/13.21
divider spanning 0-16 V, so a 5 V and a 12 V sensor both fit without
touching anything. Resolution was never the reason for a narrower range: a
5 V sensor lands at 0.836 V, which on a 16-bit ADS1115 is 6688 counts.

The real reason is the differential ground. A channel switched to 0-16 V
while the shared return attenuator stayed at the 0-5 V ratio subtracts
0.5769*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
Parts:
- added C18, C22, C23: 100nF, Capacitor_SMD:C_0805_2012Metric, symbol Device:C
- added C19: 1uF, Capacitor_SMD:C_0805_2012Metric, symbol Device:C
- added C20, C21: 15pF, Capacitor_SMD:C_0805_2012Metric, symbol Device:C
- added C24: 4.7nF, Capacitor_SMD:C_0805_2012Metric, symbol Device:C
- added D9: SMAJ26CA, Diode_SMD:D_SMA, symbol Device:D_TVS
- added JP3: TERM2 (default OFF), Jumper:SolderJumper-2_P1.3mm_Open_Pad1.0x1.5mm, symbol Jumper:SolderJumper_2_Open
- added JP4: AUXSEL (default K-line), Jumper:SolderJumper-3_P1.3mm_Bridged12_Pad1.0x1.5mm, symbol Jumper:SolderJumper_3_Bridged12
- added JP5: AUXCL (default OFF), Jumper:SolderJumper-2_P1.3mm_Open_Pad1.0x1.5mm, symbol Jumper:SolderJumper_2_Open
- added L2: 51uH, esp32autosport:L_CommonMode_TDK_ACT45B, symbol Device:L_Coupled
- added R25: 10k, Resistor_SMD:R_0805_2012Metric, symbol Device:R
- added R26, R27: 60.4, Resistor_SMD:R_0805_2012Metric, symbol Device:R
- added TP11: AUX_A, TestPoint:TestPoint_Pad_D1.5mm, symbol Connector:TestPoint
- added U6: MCP2518FD, Package_SO:SOIC-14_3.9x8.7mm_P1.27mm, symbol Interface_CAN_LIN:MCP2517FD-xSL
- added U7: TJA1051T/3, Package_SO:SOIC-8_3.9x4.9mm_P1.27mm, symbol Interface_CAN_LIN:TJA1051T-3
- added Y1: 40MHz, Crystal:Crystal_SMD_3225-4Pin_3.2x2.5mm, symbol Device:Crystal_GND24
- D7: value SMAJ26CA -> BAT54S; footprint Diode_SMD:D_SMA -> Package_TO_SOT_SMD:SOT-23; symbol Device:D_TVS -> Device:D_Schottky_Dual_Series_AKC; MPN Diodes Inc SMAJ26CA-13-F -> MDD BAT54S; Note K-line harness clamp. Same part as the two CAN clamps, so i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 -> RX clamp. This one is not optional -- it conducts on every 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
- D8: value BAT54S -> SMAJ26CA; footprint Package_TO_SOT_SMD:SOT-23 -> Diode_SMD:D_SMA; symbol Device:D_Schottky_Dual_Series_AKC -> Device:D_TVS; MPN MDD BAT54S -> Diodes Inc SMAJ26CA-13-F; Note RX clamp. This one is not optional -- it conducts on every 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 -> Aux port clamp, either mode
- R28: Note Default to normal (non-silent) mode -> Gate series resistor
- R29: value 60.4 -> 100k; Note Split termination upper half -> Holds the FET off while the MCU is in reset or the dev boar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
- R30: value 60.4 -> 33; footprint Resistor_SMD:R_0805_2012Metric -> Resistor_SMD:R_1206_3216Metric; Note Split termination lower half -> Series limit. ISO 9141-2 wants the tester's dominant below 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
- R31: value 10k -> 22k; Note Gate series resistor -> RX divider, upper leg
- R32: value 100k -> 10k; Note Holds the FET off while the MCU is in reset or the dev boar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 -> Lower leg: 9 V recessive gives 2.81 V, clear of the 2.48 V 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
- R33: value 33 -> 510; Note Series limit. ISO 9141-2 wants the tester's dominant below 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 -> The ISO 9141-2 tester pull-up value. 1206: 12 V across it w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
- R34: value 22k -> 10k; Note RX divider, upper leg -> Default to normal (non-silent) mode
- R35: value 10k -> 60.4; Note Lower leg: 9 V recessive gives 2.81 V, clear of the 2.48 V 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 -> Split termination upper half
- R36: value 510 -> 60.4; footprint Resistor_SMD:R_1206_3216Metric -> Resistor_SMD:R_0805_2012Metric; Note The ISO 9141-2 tester pull-up value. 1206: 12 V across it w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 -> Split termination lower half
Connections:
- net +3V3: now also D7.2 (K), C18.1, C19.1, C23.1, U6.14 (VDD), U7.5 (VIO); no longer D8.2 (K)
- net +5V: now also C22.1, U7.3 (VCC)
- net CAN_L: now also R27.2; no longer R30.2
- net CAN_S: now also R25.1; no longer R28.1
- net CAN_SPLIT: now also R26.2, R27.1; no longer R29.2, R30.1
- net GND: now also D7.1 (A), D8.2 (A2), R29.2, R34.2, C18.2, C19.2, C20.2, C21.2, C22.2, C23.2, C24.2, D9.2 (A2), R25.2, U6.7 (VSS), U7.2 (GND), Y1.2, Y1.4; no longer D7.2 (A2), D8.1 (A), R28.2, R35.2
- net K_LINE: now also R30.2, R31.1, JP4.1 (A); no longer D7.1 (A1), R34.1, R36.2
- net K_PU: now also R33.1; no longer R36.1
- net K_RX: now also D7.3 (common), R31.2, R32.1; no longer D8.3 (common), R34.2, R35.1
- net K_TX: now also R28.1; no longer R31.1
- net K_TX_D: now also R30.1; no longer R33.1
- net K_TX_G: now also R28.2, R29.1; no longer R31.2, R32.1
- net TERM_A: now also R26.1; no longer R29.1
- new net AUX_A: D8.1 (A1), JP4.2 (C), TP11.1
- new net AUX_B: D9.1 (A1), JP5.1 (A)
- new net CAN2H_T: L2.1, U7.7 (CANH)
- new net CAN2L_T: L2.3, U7.6 (CANL)
- new net CAN2_CS: U6.13 (~{CS})
- new net CAN2_H_C: JP3.1 (A), JP4.3 (B), L2.2
- new net CAN2_INT: U6.4 (~{INT})
- new net CAN2_L_C: JP5.2 (B), L2.4, R36.2
- new net CAN2_MISO: U6.12 (SDO)
- new net CAN2_MOSI: U6.11 (SDI)
- new net CAN2_RXD: U6.2 (RXCAN), U7.4 (RXD)
- new net CAN2_S: R34.1, U7.8 (S)
- new net CAN2_SCK: U6.10 (SCK)
- new net CAN2_SPLIT: C24.1, R35.2, R36.1
- new net CAN2_TXD: U6.1 (TXCAN), U7.1 (TXD)
- new net TERM2_A: JP3.2 (B), R35.1
- new net XTAL1: C20.1, U6.6 (OSC1), Y1.1
- new net XTAL2: C21.1, U6.5 (OSC2), Y1.3
- no-connect marks 0 -> 3
Other:
- moved on the sheet: JP2, Q3, R28, R29, R30, R31, R32, R33, R34, R35, R36, TP10
